File: ESP_Edgedevice.kicad_sch (KiCad schematic)
At the start: 12 parts, among them J1 HB9500-9.5-3P, J2 Barrier Terminal, U1 ESP8266_Lolin, U2 PZEM-004T, U4 LLC_BSS138

Commit message: added ADC, next changes are left
Parts:
- removed R1, R2: 10k, Resistor_THT:R_Axial_DIN0204_L3.6mm_D1.6mm_P5.08mm_Horizontal, symbol Device:R
- removed U1: ESP8266_Lolin, ESP8266:NodeMCU-LoLinV3, symbol esp8266-lolin:ESP8266_Lolin
- removed U2: PZEM-004T, PZEM-004T:PZEM-004T_V3, symbol PZEM-004T:PZEM-004T
- removed U4: LLC_BSS138, LLC_BSS138:LLC_BSS138, symbol LLC_BSS138:LLC_BSS138
- added C2: 100nF, symbol Device:C
- added U1: XIAO ESP32C3, XIAO_ESP32C3:xiao_esp32c3, symbol xiao_esp32c3:XIAO ESP32C3
Connections:
- net +3.3V: now also U1.12 (VCC_3V3)
- net GND: now also C2.2, U1.13 (GND)
- net RELAY_IN: now also U1.2 (D1)
- net VCC: now also C2.1, U1.14 (VUSB)
- no-connect marks 32 -> 10
Other:
- note removed: "BSS138 LLC"

Commit message: major changes made to schematics
Parts:
- added C17: 100nF X2, 275 V AC, symbol Device:C
- added F2: 25A Slow-Blow, symbol Device:Fuse
- added R17: 100R, symbol Device:R
- renumbered H2 to H1, H3 to H2, H5 to H3, J2 to J1, J1 to J2
Connections:
- net COM: now also C17.2, F2.2
- net LIVE: now also F2.1
- net NO: now also R17.1
- net D9: now reaches U1.10 (D9)
- net D10: now reaches U1.11 (D10)
- net D2: now reaches U1.3 (D2)
- net D8: now reaches U1.9 (D8)
- new net: C17.1, R17.2
- no-connect marks 10 -> 6
Other:
- added sheet voltagesensing.kicad_sch (voltagesensing.kicad_sch)
- note added: "Voltage Sensing"
- moved on the sheet: C1, C2, J1, J2, PS1, U1
