File: relay.kicad_sch (KiCad schematic)
At the start: 9 parts, among them J3 Conn_01x02_Pin, K1 SLA-05VDC-SL-C, Q1 S8050, U3 PC817X3NSZ1B

Commit message: major changes made to schematics
Parts:
- renumbered R13 to R1, R3 to R2, R4 to R3, U3 to U2
