File: voltagesensing.kicad_sch (KiCad schematic)
At the start: 19 parts, among them U4 AMS1117-5.0, U5 AMC1200SDUBR

Commit message: added ADC, next changes are left
Parts:
- added C8: 100nF, symbol Device:C
- added F1: 1A,250V AC, symbol Device:Fuse
- added RV1: Varistor, symbol Device:Varistor
- added U1: ADS131M02IPWR, TSSOP20_PW_TEX, symbol 2026-10-08_08-05-28:ADS131M02IPWR
- C1: value 470nF -> 470nF X2
- R5: value 220 -> 220R 1W
Connections:
- net GND: now also C8.1
- net GND1: now also RV1.2
- net L: now also F1.1; no longer R5.1, R7.1
- net V_OUT_N: now reaches U5.6 (VOUTN)
- net AC sensing renamed V_OUT_P
- net VCC_3.3 renamed +3.3V
- net +3.3V: now also C8.2
- new net: F1.2, R5.1, R7.1, RV1.1
- no-connect marks 1 -> 0

Commit message: major changes made to schematics
Parts:
- removed U1: ADS131M02IPWR, TSSOP20_PW_TEX, symbol 2026-10-08_08-05-28:ADS131M02IPWR
- added C10, C11, C13, C14, C16, C9: 100nF, symbol Device:C
- added J4: Conn_01x02, symbol Connector_Generic:Conn_01x02
- added R12: R, symbol Device:R
- added R13, R14, R16: 10k, symbol Device:R
- added R15: 1k, symbol Device:R
- added U5, U6: OPA333xxDBV, Package_TO_SOT_SMD:SOT-23-5, symbol Amplifier_Operational:OPA333xxDBV
- added U7: MCP3202, symbol Analog_ADC:MCP3202
- renumbered C7 to C12, C8 to C15, C1 to C3, C2 to C4, C3 to C5, C4 to C6, C5 to C7, C6 to C8, R11 to R10, R12 to R11, R5 to R4, R6 to R5, R7 to R6, R8 to R7, R9 to R8, R10 to R9, U4 to U3, U5 to U4
Connections:
- net +3.3V: now also C10.2, C16.1, C9.1, R13.1, R16.1, U5.5 (V+), U6.5 (V+), U7.8 (VDD/VREF)
- net GND: now also C10.1, C11.2, C13.2, C14.2, C16.2, C9.2, R14.2, U5.2 (V-), U6.2 (V-), U7.4 (VSS)
- net V_OUT_P: now also U5.3 (+)
- new net: C13.1, R15.2, U7.2 (CH0)
- new net: C14.1, R12.1, U7.3 (CH1)
- new net: R15.1, U5.1, U5.4 (-)
- new net: J4.2 (Pin_2), R12.2
- new net D10: U7.5 (DIN)
- new net D2: R16.2, U7.1 (~{CS}/SHDN)
- new net D8: U7.7 (CLK)
- new net D9: U7.6 (DOUT)
- new net VBIAS: C11.1, R13.2, R14.1, U6.3 (+)
- new net VBIAS_BUF: J4.1 (Pin_1), U6.1, U6.4 (-)
- no-connect marks 0 -> 1
Other:
- moved on the sheet: C12, C15, C3, C4, C5, C6, C7, C8, D3, D4, F1, R10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
