File: PCB_SHEMS/ESP_Edgedevice/ESP_Edgedevice.kicad_sch (KiCad schematic)
At the start: 9 parts, among them J3 Conn_01x02_Pin, K1 SLA-05VDC-SL-C, Q1 S8050, U2 PC817X3NSZ1B

Commit message: PCB left
Parts:
- removed D1: LED, LED_THT:LED_D3.0mm, symbol Device:LED
- removed D2: 1N4007, Diode_THT:D_DO-41_SOD81_P10.16mm_Horizontal, symbol Diode:1N4007
- removed J3: Conn_01x02_Pin, Connector_PinHeader_2.54mm:PinHeader_1x02_P2.54mm_Vertical, symbol Connector:Conn_01x02_Pin
- removed K1: SLA-05VDC-SL-C, SLA_05VDC_SL_C:K_SLA_C_NFR, symbol SLA-05VDC-SL-C:SLA-05VDC-SL-C
- removed Q1: S8050, Package_TO_SOT_THT:TO-92_Inline_Wide, symbol Transistor_BJT:S8050
- removed R1, R3: 1K, Resistor_THT:R_Axial_DIN0207_L6.3mm_D2.5mm_P10.16mm_Horizontal, symbol Device:R
- removed R2: 2.2K, Resistor_THT:R_Axial_DIN0207_L6.3mm_D2.5mm_P10.16mm_Horizontal, symbol Device:R
- removed U2: PC817X3NSZ1B, Connector_PinHeader_2.54mm:PinHeader_1x04_P2.54mm_Vertical, symbol PC817X3NSZ1B:PC817X3NSZ1B
- added C1: 470uF, Capacitor_THT:CP_Radial_D6.3mm_P2.50mm, symbol Device:C_Polarized
- added C17: 100nF X2, 275 V AC, Capacitor_THT:C_Rect_L18.0mm_W5.0mm_P15.00mm_FKS3_FKP3, symbol Device:C
- added F2: 25A Slow-Blow, Fuse:Fuseholder_Cylinder-6.3x32mm_Schurter_0031-8002_Horizontal_Open, symbol Device:Fuse
- added H1, H2, H3: MountingHole, MountingHole:MountingHole_2.1mm, symbol Mechanical:MountingHole
- added J1: Barrier Terminal, Connector_Phoenix_MSTB:PhoenixContact_MSTBA_2,5_2-G_1x02_P5.00mm_Horizontal, symbol SparkFun-Connector:Barrier_Terminal_9.5mm-2
- added J2: HB9500-9.5-3P, Connector_Phoenix_MSTB:PhoenixContact_MSTBA_2,5_3-G_1x03_P5.00mm_Horizontal, symbol HB9500-9.5-3P:HB9500-9.5-3P
- added PS1: HLK-5M05, Converter_ACDC:Converter_ACDC_Hi-Link_HLK-5Mxx, symbol Converter_ACDC:HLK-5M05
- added R17: 100R, Resistor_THT:R_Axial_DIN0309_L9.0mm_D3.2mm_P12.70mm_Horizontal, symbol Device:R
- added U1: XIAO ESP32C3, xiao-esp32-c3:xiao_esp32c3, symbol xiao_esp32c3:XIAO ESP32C3
Connections:
- net COM: now also C17.2, F2.2, J2.2
- net GND: now also C1.2, PS1.3 (-Vout), U1.13 (GND)
- net NC: now also J2.3
- net NO: now also J2.1, R17.1
- net VCC: now also C1.1, PS1.4 (+Vout), U1.14 (VUSB)
- new net: C17.1, R17.2
- new net +3.3V: U1.12 (VCC_3V3)
- new net D10: U1.11 (D10)
- new net D2: U1.3 (D2)
- new net D8: U1.9 (D8)
- new net D9: U1.10 (D9)
- new net LIVE: F2.1, J1.2 (Pin_2), PS1.1 (AC/L)
- new net NEUTRAL: J1.1 (Pin_1), PS1.2 (AC/N)
- new net RELAY_IN: U1.2 (D1)
- no-connect marks 0 -> 8
Other:
- added sheet Relay (relay.kicad_sch)
- added sheet voltagesensing.kicad_sch (voltagesensing.kicad_sch)
- note added: "Hilink 5v/5W powersupply"
- note added: "Relay part"
- note added: "Voltage Sensing"
- title: Relay -> ${project_name}

Commit message: more changes midnight
Parts:
- added H4: MountingHole, MountingHole:MountingHole_2.1mm, symbol Mechanical:MountingHole
Changed lines of the file:
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@@
+		)
+	)
+	(symbol
+		(lib_id "Mechanical:MountingHole")
+		(at 157.48 189.23 0)
+		(unit 1)
+		(body_style 1)
+		(exclude_from_sim no)
+		(in_bom no)
+		(on_board yes)
+		(in_pos_files yes)
+		(dnp no)
+		(fields_autoplaced yes)
+		(property "Reference" "H4"
+			(at 160.02 187.9599 0)
+			(show_name no)
+			(do_not_autoplace no)
+			(effects
+				(font
+					(size 1.27 1.27)
+				)
+				(justify left)
+			)
+		)
+		(property "Value" "MountingHole"
+			(at 160.02 190.4999 0)
+			(show_name no)
+			(do_not_autoplace no)
+			(effects
+				(font
+					(size 1.27 1.27)
+				)
+				(justify left)
+			)
+		)
+		(property "Footprint" "MountingHole:MountingHole_2.1mm"
+			(at 157.48 189.23 0)
+			(hide yes)
+			(show_name no)
+			(do_not_autoplace no)
+			(effects
+				(font
+					(size 1.27 1.27)
+				)
+			)
+		)
+		(property "Datasheet" ""
+			(at 157.48 189.23 0)
+			(hide yes)
+			(show_name no)
+			(do_not_autoplace no)
+			(effects
+				(font
+					(size 1.27 1.27)
+				)
+			)
+		)
+		(property "Description" "Mounting Hole without connection"
+			(at 157.48 189.23 0)
+			(hide yes)
+			(show_name no)
+			(do_not_autoplace no)
+			(effects
+				(font
+					(size 1.27 1.27)
+				)
+			)
+		)
+		(instances
+			(project "ESP_Edgedevice"
+				(path "/8fa9f2a2-260d-4024-b3c1-a0bc52ef0867"
+					(reference "H4")
+					(unit 1)
+				)
+			)
 		)
 	)

Commit message: made more Schema changes in Lab
Parts:
- J2: footprint Connector_Phoenix_MSTB:PhoenixContact_MSTBA_2,5_3-G_1x03_P5.00mm_Horizontal -> myparts:HB9500_9.5-3P
- U1: footprint xiao-esp32-c3:xiao_esp32c3 -> myparts:XIAO_Socket_W15.24
Changed lines of the file:
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@@
 			)
 		)
-		(property "Footprint" "xiao-esp32-c3:xiao_esp32c3"
+		(property "Footprint" "myparts:XIAO_Socket_W15.24"
 			(at 130.81 16.51 0)
 			(hide yes)
@@
 			)
 		)
-		(property "Footprint" "Connector_Phoenix_MSTB:PhoenixContact_MSTBA_2,5_3-G_1x03_P5.00mm_Horizontal"
+		(property "Footprint" "myparts:HB9500_9.5-3P"
 			(at 250.19 22.86 0)
 			(hide yes)
