File: PCB_SHEMS/ESP_Edgedevice/relay.kicad_sch (KiCad schematic)
At the start: 12 parts, among them J1 Barrier Terminal, J2 HB9500-9.5-3P, U1 XIAO ESP32C3

Commit message: PCB left
Parts:
- removed C1: 470uF, Capacitor_THT:CP_Radial_D6.3mm_P2.50mm, symbol Device:C_Polarized
- removed C17: 100nF X2, 275 V AC, symbol Device:C
- removed C2: 100nF, symbol Device:C
- removed F2: 25A Slow-Blow, symbol Device:Fuse
- removed H1, H2, H3: MountingHole, MountingHole:MountingHole_2.1mm, symbol Mechanical:MountingHole
- removed J1: Barrier Terminal, Connector_Phoenix_MSTB:PhoenixContact_MSTBA_2,5_2-G_1x02_P5.00mm_Horizontal, symbol SparkFun-Connector:Barrier_Terminal_9.5mm-2
- removed J2: HB9500-9.5-3P, Connector_Phoenix_MSTB:PhoenixContact_MSTBA_2,5_3-G_1x03_P5.00mm_Horizontal, symbol HB9500-9.5-3P:HB9500-9.5-3P
- removed PS1: HLK-5M05, Converter_ACDC:Converter_ACDC_Hi-Link_HLK-5Mxx, symbol Converter_ACDC:HLK-5M05
- removed R17: 100R, symbol Device:R
- removed U1: XIAO ESP32C3, XIAO_ESP32C3:xiao_esp32c3, symbol xiao_esp32c3:XIAO ESP32C3
- added D1: LED, LED_THT:LED_D3.0mm, symbol Device:LED
- added D2: 1N4007, Diode_THT:D_DO-41_SOD81_P10.16mm_Horizontal, symbol Diode:1N4007
- added J3: Conn_01x02_Pin, Connector_PinHeader_2.54mm:PinHeader_1x02_P2.54mm_Vertical, symbol Connector:Conn_01x02_Pin
- added K1: SLA-05VDC-SL-C, SLA-05VDC-SL-C:RELAY-TH_SLA-XXVDC-XX-C, symbol SLA-05VDC-SL-C:SLA-05VDC-SL-C
- added Q1: S8050, Package_TO_SOT_THT:TO-92_Inline_Wide, symbol Transistor_BJT:S8050
- added R1, R3: 1K, Resistor_THT:R_Axial_DIN0207_L6.3mm_D2.5mm_P10.16mm_Horizontal, symbol Device:R
- added R2: 2.2K, Resistor_THT:R_Axial_DIN0207_L6.3mm_D2.5mm_P10.16mm_Horizontal, symbol Device:R
- added U2: PC817X3NSZ1B, Package_DIP:DIP-4_W7.62mm, symbol PC817X3NSZ1B:PC817X3NSZ1B
Connections:
- net COM: now also K1.3, K1.4
- net GND: now also Q1.1 (E), R1.2, U2.2
- net NC: now also K1.6
- net NO: now also K1.5
- net VCC: now also J3.2 (Pin_2)
- new net: D1.1 (K), R1.1
- new net: R3.1, U2.3
- new net: Q1.2 (B), R3.2
- new net: R2.2, U2.1
- new net INPUT: D1.2 (A), R2.1
- new net Jd_VCC: D2.1 (K), J3.1 (Pin_1), K1.1, U2.4
- new net Relay: D2.2 (A), K1.2, Q1.3 (C)
- no-connect marks 6 -> 0
Other:
- removed sheet Relay
- removed sheet voltagesensing.kicad_sch
- note removed: "Hilink 5v/5W powersupply"
- note removed: "Relay part"
- note removed: "Voltage Sensing"
- title: ${project_name} -> Relay

Commit message: made more Schema changes in Lab
Parts:
- R1, R3: footprint Resistor_THT:R_Axial_DIN0207_L6.3mm_D2.5mm_P10.16mm_Horizontal -> Resistor_SMD:R_1206_3216Metric
- R2: value 2.2K -> 1k; footprint Resistor_THT:R_Axial_DIN0207_L6.3mm_D2.5mm_P10.16mm_Horizontal -> Resistor_SMD:R_1206_3216Metric
