File: PCB_SHEMS/ESP_Edgedevice/voltagesensing.kicad_sch (KiCad schematic)
At the start: 37 parts, among them J4 Conn_01x02, U3 AMS1117-5.0, U4 AMC1200SDUBR, U5 OPA333xxDBV, U6 OPA333xxDBV, U7 MCP3202

Commit message: PCB left
Parts:
- removed C12: 10uF, Capacitor_THT:CP_Radial_D5.0mm_P2.50mm, symbol Device:C_Polarized_US
- C10, C11, C13, C14, C15: footprint (none) -> Capacitor_THT:C_Disc_D5.0mm_W2.5mm_P5.00mm
- C16, C9: footprint (none) -> Capacitor_SMD:C_0805_2012Metric
- C3: footprint capacitor:CAP_150AXIAL_RF_CND -> Capacitor_THT:C_Rect_L26.5mm_W8.5mm_P22.50mm_MKS4
- C5: footprint Capacitor_SMD:C_1206_3216Metric_Pad1.33x1.80mm_HandSolder -> Capacitor_THT:CP_Radial_D10.0mm_P5.00mm
- C6: footprint Capacitor_SMD:C_1206_3216Metric_Pad1.33x1.80mm_HandSolder -> Capacitor_THT:C_Disc_D5.0mm_W2.5mm_P5.00mm
- C8: footprint Capacitor_SMD:C_1206_3216Metric -> Capacitor_THT:C_Disc_D5.0mm_W2.5mm_P5.00mm
- F1: footprint (none) -> Fuse:Fuseholder_Cylinder-5x20mm_Schurter_0031_8201_Horizontal_Open
- J4: footprint (none) -> Connector_PinHeader_2.54mm:PinHeader_1x02_P2.54mm_Vertical
- R12: value R -> 1k; footprint (none) -> Resistor_THT:R_Axial_DIN0207_L6.3mm_D2.5mm_P10.16mm_Horizontal
- R13, R14, R15, R16: footprint (none) -> Resistor_THT:R_Axial_DIN0207_L6.3mm_D2.5mm_P10.16mm_Horizontal
- RV1: footprint (none) -> Varistor:RV_Disc_D12mm_W4.2mm_P7.5mm
- U7: footprint (none) -> Package_SO:TSSOP-8_3x3mm_P0.65mm
Other:
- title: (none) -> Voltage Sensing
- moved on the sheet: C15

Commit message: made more Schema changes in Lab
Parts:
- C10, C11, C13, C14, C15, C8: footprint Capacitor_THT:C_Disc_D5.0mm_W2.5mm_P5.00mm -> Capacitor_SMD:C_1206_3216Metric
- C16, C9: footprint Capacitor_SMD:C_0805_2012Metric -> Capacitor_SMD:C_1206_3216Metric
- C5: footprint Capacitor_THT:CP_Radial_D10.0mm_P5.00mm -> Capacitor_SMD:C_1206_3216Metric
- C6: footprint Capacitor_THT:C_Disc_D5.0mm_W2.5mm_P5.00mm -> Capacitor_THT:CP_Radial_D5.0mm_P2.50mm
- R10, R11, R12, R13, R14, R15, R16, R8, R9: footprint Resistor_THT:R_Axial_DIN0207_L6.3mm_D2.5mm_P10.16mm_Horizontal -> Resistor_SMD:R_1206_3216Metric
- U7: footprint Package_SO:TSSOP-8_3x3mm_P0.65mm -> Package_SO:TSSOP-8_4.4x3mm_P0.65mm
Other:
- moved on the sheet: C10, C11, C13, C14, C16, C9, J4, R12, R13, R14, R15, R16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
